Commit message: Complete the slam map

File: src/vacuum_describe/urdf/vacuum.urdf (robot description, URDF)
Before this commit: robot vacuum_cleaner, 3 links, 2 joints
Joints:
- joint imu_joint: origin xyz=0.0 0.0 0.05 rpy=0 0 0 -> xyz=0.05 0.0 0.05 rpy=0 0 0
- joint lidar_joint: origin xyz=0.1 0.0 0.08 rpy=0 0 0 -> xyz=0.12 0.0 0.08 rpy=0 0 -1.5708

Commit message: backup

File: src/vacuum_describe/urdf/vacuum.urdf (robot description, URDF)
Before this commit: robot vacuum_cleaner, 4 links, 3 joints
Links:
- removed link base_footprint
Joints:
- removed joint base_joint
- joint lidar_joint: origin xyz=0.12 0.0 0.08 rpy=0 0 -1.5708 -> xyz=0.0 -0.1 0.1 rpy=0 0 0

Commit message: backup and Claude will help me ((wish

File: src/vacuum_describe/urdf/vacuum.urdf (robot description, URDF)
Before this commit: robot vacuum_cleaner, 3 links, 2 joints
Joints:
- joint lidar_joint: origin xyz=0.0 -0.1 0.1 rpy=0 0 0 -> xyz=0.0 -0.1 0.1 rpy=0 0 -3.1416
